Commit message: 21_02_25

File: xacro/model/spotdog.xacro (robot description, xacro)
@@ -6,4 +6,5 @@
     <xacro:include filename="$(find spotdog)/xacro/transmission/transmission.xacro"/>
     <xacro:base_link name="BASE"/>
+<!--
     <link name="dummy_link"/>
     <joint name="base_to_dummy_link" type="fixed">
@@ -11,5 +12,5 @@
         <child link="BASE"/>
         <origin xyz="0.0 0.0 1" rpy="0.0 0.0 0.0"/>
-    </joint>
+    </joint> -->
     <!-- <link name="world"/>
     <joint name="world_to_base" type="fixed">
@@ -68,23 +69,23 @@
         </joint>
     </gazebo>
-    <xacro:transmission name="FR_hip_trans" joint_name="base_to_fr_upper_hip" actuator_name="trans_1"/>
-    <xacro:transmission name="BR_hip_trans" joint_name="base_to_br_upper_hip" actuator_name="trans_2"/>
-    <xacro:transmission name="FL_hip_trans" joint_name="base_to_fl_upper_hip" actuator_name="trans_3"/>
-    <xacro:transmission name="BL_hip_trans" joint_name="base_to_bl_upper_hip" actuator_name="trans_4"/>
-    <xacro:transmission name="FR_knee_trans" joint_name="base_to_fr_upper_knee" actuator_name="trans_5"/>
-    <xacro:transmission name="BR_knee_trans" joint_name="base_to_br_upper_knee" actuator_name="trans_6"/>
-    <xacro:transmission name="FL_knee_trans" joint_name="base_to_fl_upper_knee" actuator_name="trans_7"/>
-    <xacro:transmission name="BL_knee_trans" joint_name="base_to_bl_upper_knee" actuator_name="trans_8"/>
-    <xacro:transmission name="FR_upper_hip_to_lower_hip_trans" joint_name="FR_upper_hip_to_lower_hip" actuator_name="trans_9"/>
-    <xacro:transmission name="BR_upper_hip_to_lower_hip_trans" joint_name="BR_upper_hip_to_lower_hip" actuator_name="trans_10"/>
-    <xacro:transmission name="FL_upper_hip_to_lower_hip_trans" joint_name="FL_upper_hip_to_lower_hip" actuator_name="trans_11"/>
-    <xacro:transmission name="BL_upper_hip_to_lower_hip_trans" joint_name="BL_upper_hip_to_lower_hip" actuator_name="trans_12"/>
-    <xacro:transmission name="FR_upper_knee_to_lower_knee_trans" joint_name="FR_upper_knee_to_lower_knee" actuator_name="trans_13"/>
-    <xacro:transmission name="BR_upper_knee_to_lower_knee_trans" joint_name="BR_upper_knee_to_lower_knee" actuator_name="trans_14"/>
-    <xacro:transmission name="FL_upper_knee_to_lower_knee_trans" joint_name="FL_upper_knee_to_lower_knee" actuator_name="trans_15"/>
-    <xacro:transmission name="BL_upper_knee_to_lower_knee_trans" joint_name="BL_upper_knee_to_lower_knee" actuator_name="trans_16"/>
+    <xacro:transmissionEffortJoint name="FR_hip_trans" joint_name="base_to_fr_upper_hip" actuator_name="trans_1"/>
+    <xacro:transmissionEffortJoint name="BR_hip_trans" joint_name="base_to_br_upper_hip" actuator_name="trans_2"/>
+    <xacro:transmissionEffortJoint name="FL_hip_trans" joint_name="base_to_fl_upper_hip" actuator_name="trans_3"/>
+    <xacro:transmissionEffortJoint name="BL_hip_trans" joint_name="base_to_bl_upper_hip" actuator_name="trans_4"/>
+    <xacro:transmissionPassiveJoint name="FR_knee_trans" joint_name="base_to_fr_upper_knee" actuator_name="trans_5"/>
+    <xacro:transmissionPassiveJoint name="BR_knee_trans" joint_name="base_to_br_upper_knee" actuator_name="trans_6"/>
+    <xacro:transmissionPassiveJoint name="FL_knee_trans" joint_name="base_to_fl_upper_knee" actuator_name="trans_7"/>
+    <xacro:transmissionPassiveJoint name="BL_knee_trans" joint_name="base_to_bl_upper_knee" actuator_name="trans_8"/>
+    <xacro:transmissionPassiveJoint name="FR_upper_hip_to_lower_hip_trans" joint_name="FR_upper_hip_to_lower_hip" actuator_name="trans_9"/>
+    <xacro:transmissionPassiveJoint name="BR_upper_hip_to_lower_hip_trans" joint_name="BR_upper_hip_to_lower_hip" actuator_name="trans_10"/>
+    <xacro:transmissionPassiveJoint name="FL_upper_hip_to_lower_hip_trans" joint_name="FL_upper_hip_to_lower_hip" actuator_name="trans_11"/>
+    <xacro:transmissionPassiveJoint name="BL_upper_hip_to_lower_hip_trans" joint_name="BL_upper_hip_to_lower_hip" actuator_name="trans_12"/>
+    <xacro:transmissionPassiveJoint name="FR_upper_knee_to_lower_knee_trans" joint_name="FR_upper_knee_to_lower_knee" actuator_name="trans_13"/>
+    <xacro:transmissionPassiveJoint name="BR_upper_knee_to_lower_knee_trans" joint_name="BR_upper_knee_to_lower_knee" actuator_name="trans_14"/>
+    <xacro:transmissionPassiveJoint name="FL_upper_knee_to_lower_knee_trans" joint_name="FL_upper_knee_to_lower_knee" actuator_name="trans_15"/>
+    <xacro:transmissionPassiveJoint name="BL_upper_knee_to_lower_knee_trans" joint_name="BL_upper_knee_to_lower_knee" actuator_name="trans_16"/>
     <gazebo>
         <plugin name='gazebo_ros_control' filename= 'libgazebo_ros_control.so'>
-          <robotNamespace>/spotdog</robotNamespace>
+          <robotNamespace>/</robotNamespace>
           <robotSimType>gazebo_ros_control/ClosedLoopHWSim</robotSimType>
         </plugin>

File: xacro/transmission/transmission.xacro (robot description, xacro)
@@ -1,5 +1,5 @@
 <?xml version="1.0"?>
 <robot xmlns:xacro="http://www.ros.org/wiki/xacro">
-    <xacro:macro name="transmission" params="name joint_name actuator_name">
+    <xacro:macro name="transmissionPassiveJoint" params="name joint_name actuator_name">
         <transmission name="${name}">
             <type>transmission_interface/SimpleTransmission</type>
@@ -13,3 +13,15 @@
         </transmission>
     </xacro:macro>
+    <xacro:macro name="transmissionEffortJoint" params="name joint_name actuator_name">
+        <transmission name="${name}">
+            <type>transmission_interface/SimpleTransmission</type>
+            <joint name="${joint_name}">
+                <hardwareInterface>hardware_interface/EffortJointInterface</hardwareInterface>
+            </joint>
+            <actuator name="${actuator_name}">
+                <mechanicalReduction>1.0</mechanicalReduction>
+                <hardwareInterface>hardware_interface/EffortJointInterface</hardwareInterface>
+            </actuator>
+        </transmission>
+    </xacro:macro>
 </robot>
